Commit message: Integrates Ridgeback URDF with Baxter's Xacro URDF
- Adds a ridgeback_baxter_world.launch to demonstrate how to launch
  the Ridgeback with Baxter in Gazebo (this needs some Ridgeback tweaks)
- Adds a pedestal stand segment and DAE's for combining the two platforms
- Makes Baxter's Torso the parent of the Ridgeback for integrating with
  Baxter's onboard mutable robot state publisher
- Makes Baxter model optional to allow for publishing the
  Ridgeback-Pedestal combo as a URDF fragment for the real Baxter:
  $ rosrun xacro xacro.py --inorder
    `rospack find ridgeback_baxter_description`/urdf/ridgeback_baxter.urdf.xacro
     with_baxter:=false  > ridgeback_baxter.xml
  # After making ridgeback_baxter.yaml with the following values:
  # time: current time
  # link: 'torso'
  # joint: 'pedestal_fixed'
  # urdf: xml from ridgeback_baxter.xml
  $ rostopic pub /robot/urdf baxter_core_msgs/URDFConfiguration -f ridgeback_baxter.yaml -l
  # The real robot will replace its pedestal with the URDF fragment that you just created
  # (you will likely then want to publish your wheel joint states to /robot/joint_states)
- Enjoy the marvels of your new mobile Baxter!

File: ridgeback_baxter_description/urdf/ridgeback_baxter.urdf.xacro (robot description, xacro)
@@ -1,13 +1,51 @@
 <?xml version="1.0"?>
 <robot name="ridgeback_baxter" xmlns:xacro="http://www.ros.org/wiki/xacro">
-  <xacro:property name="pedestal_height" value="0.565" />
+  <xacro:arg name="gazebo" default="false"/>
+  <xacro:arg name="pedestal" default="false"/>
+  <xacro:arg name="with_baxter" default="true"/>
+  <xacro:property name="pedestal_height" value="-0.92" />
   <xacro:property name="pedestal_diameter" value="0.203" />
-  <xacro:property name="pedestal_offset_x" value="0.2" />
+  <xacro:property name="pedestal_offset_x" value="-0.2" />
+  <!-- Ridgeback URDF -->
   <xacro:include filename="$(find ridgeback_description)/urdf/ridgeback.urdf.xacro" />
-  <xacro:include filename="$(find baxter_description)/urdf/baxter.urdf" />
-  <joint name="ridgeback_base_to_baxter" type="fixed">
+  <xacro:if value="$(arg with_baxter)">
+    <!-- Baxter URDF -->
+    <xacro:include filename="$(find baxter_description)/urdf/baxter.urdf.xacro">
+      <xacro:arg name="gazebo" value="${gazebo}"/>
+      <xacro:arg name="pedestal" value="${pedestal}"/>
+    </xacro:include>
+  </xacro:if>
+  <!-- Ridgeback-Baxter Joint URDF -->
+  <joint name="pedestal_fixed" type="fixed">
+    <origin rpy="0 0 0" xyz="0 0 0" />
+    <parent link="torso" />
+    <child link="pedestal_stand" />
+  </joint>
+  <link name="pedestal_stand">
+    <visual>
+      <origin rpy="0 0 0" xyz="0 0 0"/>
+      <geometry>
+        <mesh filename="package://ridgeback_baxter_description/meshes/pedestal_stand.dae"/>
+      </geometry>
+      <material name="darkgray">
+        <color rgba=".2 .2 .2 1"/>
+      </material>
+    </visual>
+    <collision>
+      <origin rpy="0 0 0" xyz="0 0 0"/>
+      <geometry>
+        <mesh filename="package://ridgeback_baxter_description/meshes/pedestal_stand_collision.dae"/>
+      </geometry>
+    </collision>
+    <inertial>
+      <origin rpy="0 0 0" xyz="0 0 0"/>
+      <mass value="30.0"/>
+      <inertia ixx="5.0635929" ixy="0.00103417" ixz="0.80199628" iyy="6.08689388" iyz="0.00105311" izz="4.96191932"/>
+    </inertial>
+  </link>
+  <joint name="baxter_to_ridgeback_base" type="fixed">
     <origin rpy="0 0 0" xyz="${pedestal_offset_x} 0 ${pedestal_height}" />
-    <parent link="mid_mount" />
-    <child link="base" />
+    <parent link="pedestal_stand" />
+    <child link="base_link" />
   </joint>
 </robot>
